Commit message: Done lab 3

File: src/exercise_3_4/description/colours.xacro (robot description, xacro)
@@ -16,3 +16,9 @@
         <color rgba="0 0 0 1"/>
     </material>
+    <material name="magenta">
+        <color rgba="1 0 1 1"/>
+    </material>
+    <material name="red">
+        <color rgba="1 0 0 1"/>
+    </material>
 </robot>

File: src/lab2urdf/description/gazebo.xacro (robot description, xacro)
@@ -25,4 +25,6 @@
             name="ignition::gazebo::systems::JointStatePublisher">
         </plugin>
+    </gazebo>
+    <gazebo>
         <plugin
             filename="libignition-gazebo-odometry-publisher-system"
