Commit message: everything but 4_5 done

File: src/lab04/description/robot.urdf (robot description, URDF)
Before this commit: robot robot, 6 links, 5 joints
Links:
- added link camera_link; visual box size=0.010 0.03 0.03
- added link camera_link_optical
Joints:
- added joint camera_joint: type fixed, parent chassis, child camera_link, origin xyz=0.305 0 0.08 rpy=0 0 0
- added joint camera_optical_joint: type fixed, parent camera_link, child camera_link_optical, origin xyz=0 0 0 rpy=-1.5707963267948966 0 -1.5707963267948966

File: src/lab04/description/robot.urdf.xacro (robot description, xacro)
@@ -16,3 +16,4 @@
     <xacro:include filename="robot_core.xacro" />
     <xacro:include filename="lidar.xacro" />
+    <xacro:include filename="camera.xacro" />
 </robot>
