Commit message: starting excersice 4.1

File: src/lab04/description/colors.xacro (robot description, xacro)
@@ -7,4 +7,7 @@
         <color rgba="1 0.3 0.1 1"/>
     </material>
+    <material name="green">
+        <color rgba="0 1 0 1"/>
+    </material>
     <material name="blue">
         <color rgba="0.2 0.2 1 1"/>
@@ -13,3 +16,9 @@
         <color rgba="0 0 0 1"/>
     </material>
+    <material name="magenta">
+        <color rgba="1 0 1 1"/>
+    </material>
+    <material name="red">
+        <color rgba="1 0 0 1"/>
+    </material>
 </robot>

File: src/lab04/description/robot.urdf.xacro (robot description, xacro)
@@ -1,4 +1,17 @@
 <?xml version="1.0"?>
 <robot xmlns:xacro="http://www.ros.org/wiki/xacro"  name="robot">
+    <xacro:property name="chassis_offset" value="-0.1" />
+    <xacro:property name="chassis_width" value="0.3" />
+    <xacro:property name="chassis_height" value="0.15" />
+    <xacro:property name="chassis_length" value="0.3" />
+    <xacro:property name="wheel_offset" value="0.175" />
+    <xacro:property name="wheel_radius" value="0.05" />
+    <xacro:property name="wheel_thickness" value="0.04" />
+    <xacro:property name="caster_offset" value="0.24" />
+    <xacro:property name="caster_radius" value="0.05" />
+    <xacro:property name="lidar_radius" value="0.05" />
+    <xacro:property name="lidar_height" value="0.04" />
+    <xacro:include filename="inertial.xacro" />
+    <xacro:include filename="gazebo.xacro" />
     <xacro:include filename="robot_core.xacro" />
     <xacro:include filename="lidar.xacro" />

File: src/lab04/description/robot_core.xacro (robot description, xacro)
@@ -29,5 +29,5 @@
                 <box size="${chassis_w} ${chassis_l} ${chassis_h}"/>
             </geometry>
-            <material name="white"/>
+            <material name="green"/>
         </visual>
         <collision>

Commit message: lab exam q1 done and q3 started

File: src/lab04/description/colors.xacro (robot description, xacro)
@@ -11,5 +11,5 @@
     </material>
     <material name="blue">
-        <color rgba="0.2 0.2 1 1"/>
+        <color rgba="0 0 1 1"/>
     </material>
     <material name="black">

File: src/lab04/description/robot.urdf (robot description, URDF)
Before this commit: robot robot, 8 links, 7 joints
Links:
- removed link caster_wheel
- removed link laser_frame
- added link left_wheel1, mass 0.1; collision cylinder length=0.1 radius=0.2; visual cylinder length=0.1 radius=0.2
- added link right_wheel1, mass 0.1; collision cylinder length=0.1 radius=0.2; visual cylinder length=0.1 radius=0.2
- added link robo_hub, mass 0.5; collision box size=0.3 0.4 0.2; visual box size=0.3 0.4 0.2
- link chassis: geometry collision box size=1.0 0.4 0.2; visual box size=1.0 0.4 0.2
- link left_wheel: geometry collision cylinder length=0.1 radius=0.2; visual cylinder length=0.1 radius=0.2
- link right_wheel: geometry collision cylinder length=0.1 radius=0.2; visual cylinder length=0.1 radius=0.2
Joints:
- removed joint caster_wheel_joint
- removed joint laser_joint
- added joint left_wheel_joint1: type continuous, parent base_link, child left_wheel1, origin xyz=-0.25 0.25 0.2 rpy=-1.5707963267948966 0 0, axis 0 0 1
- added joint right_wheel_joint1: type continuous, parent base_link, child right_wheel1, origin xyz=-0.25 -0.25 0.2 rpy=1.5707963267948966 0 0, axis 0 0 -1
- added joint robo_hub_joint: type fixed, parent base_link, child robo_hub, origin xyz=0 0 0
- joint chassis_joint: origin xyz=-0.1 0 0 -> xyz=0 0 0
- joint left_wheel_joint: origin xyz=0 0.175 0 rpy=-1.5707963267948966 0 0 -> xyz=0.3 0.25 0.2 rpy=-1.5707963267948966 0 0
- joint right_wheel_joint: origin xyz=0 -0.175 0 rpy=1.5707963267948966 0 0 -> xyz=0.3 -0.25 0.2 rpy=1.5707963267948966 0 0

File: src/lab04/description/robot.urdf.xacro (robot description, xacro)
@@ -10,10 +10,7 @@
     <xacro:property name="caster_offset" value="0.24" />
     <xacro:property name="caster_radius" value="0.05" />
-    <xacro:property name="lidar_radius" value="0.05" />
-    <xacro:property name="lidar_height" value="0.04" />
     <xacro:include filename="inertial.xacro" />
     <xacro:include filename="gazebo.xacro" />
     <xacro:include filename="robot_core.xacro" />
-    <xacro:include filename="lidar.xacro" />
     <xacro:include filename="camera.xacro" />
 </robot>

File: src/lab04/description/robot_core.xacro (robot description, xacro)
@@ -5,5 +5,5 @@
     <link name="base_link">
     </link>
-    <xacro:property name="chassis_joint_x" value="-0.1"/>
+    <xacro:property name="chassis_joint_x" value="0"/>
     <xacro:property name="chassis_joint_y" value="0"/>
     <xacro:property name="chassis_joint_z" value="0"/>
@@ -13,10 +13,10 @@
         <origin xyz="${chassis_joint_x} ${chassis_joint_y} ${chassis_joint_z}"/>
     </joint>
-    <xacro:property name="chassis_x" value="0.15"/>
+    <xacro:property name="chassis_x" value="0"/>
     <xacro:property name="chassis_y" value="0"/>
-    <xacro:property name="chassis_z" value="0.075"/>
-    <xacro:property name="chassis_w" value="0.3"/>
-    <xacro:property name="chassis_l" value="0.3"/>
-    <xacro:property name="chassis_h" value="0.15"/>
+    <xacro:property name="chassis_z" value="0.2"/>
+    <xacro:property name="chassis_w" value="1.0"/>
+    <xacro:property name="chassis_l" value="0.4"/>
+    <xacro:property name="chassis_h" value="0.2"/>
     <xacro:property name="chassis_roll" value="0"/>
     <xacro:property name="chassis_pitch" value="0"/>
@@ -29,5 +29,5 @@
                 <box size="${chassis_w} ${chassis_l} ${chassis_h}"/>
             </geometry>
-            <material name="green"/>
+            <material name="blue"/>
         </visual>
         <collision>
@@ -42,7 +42,7 @@
     </link>
     <!-- LEFT WHEEL -->
-    <xacro:property name="l_wheel_joint_x" value="0"/>
-    <xacro:property name="l_wheel_joint_y" value="0.175"/>
-    <xacro:property name="l_wheel_joint_z" value="0"/>
+    <xacro:property name="l_wheel_joint_x" value="0.3"/>
+    <xacro:property name="l_wheel_joint_y" value="0.25"/>
+    <xacro:property name="l_wheel_joint_z" value="0.2"/>
     <xacro:property name="l_wheel_joint_ax" value="0"/>
     <xacro:property name="l_wheel_joint_ay" value="0"/>
@@ -57,6 +57,6 @@
         <axis xyz="${l_wheel_joint_ax} ${l_wheel_joint_ay} ${l_wheel_joint_az}"/>
     </joint>
-    <xacro:property name="l_wheel_length" value="0.04"/>
-    <xacro:property name="l_wheel_radius" value="0.05"/>
+    <xacro:property name="l_wheel_length" value="0.1"/>
+    <xacro:property name="l_wheel_radius" value="0.2"/>
     <xacro:property name="l_wheel_m" value="0.1"/>
     <xacro:property name="l_wheel_x" value="0"/>
@@ -71,5 +71,5 @@
                 <cylinder length="${l_wheel_length}" radius="${l_wheel_radius}"/>
             </geometry>
-            <material name="blue"/>
+            <material name="red"/>
         </visual>
         <collision>
@@ -83,7 +83,7 @@
     </link>
     <!-- RIGHT WHEEL -->
-    <xacro:property name="r_wheel_joint_x" value="0"/>
-    <xacro:property name="r_wheel_joint_y" value="-0.175"/>
-    <xacro:property name="r_wheel_joint_z" value="0"/>
+    <xacro:property name="r_wheel_joint_x" value="0.3"/>
+    <xacro:property name="r_wheel_joint_y" value="-0.25"/>
+    <xacro:property name="r_wheel_joint_z" value="0.2"/>
     <xacro:property name="r_wheel_joint_ax" value="0"/>
     <xacro:property name="r_wheel_joint_ay" value="0"/>
@@ -98,6 +98,6 @@
         <axis xyz="${r_wheel_joint_ax} ${r_wheel_joint_ay} ${r_wheel_joint_az}"/>
     </joint>
-    <xacro:property name="r_wheel_length" value="0.04"/>
-    <xacro:property name="r_wheel_radius" value="0.05"/>
+    <xacro:property name="r_wheel_length" value="0.1"/>
+    <xacro:property name="r_wheel_radius" value="0.2"/>
     <xacro:property name="r_wheel_m" value="0.1"/>
     <xacro:property name="r_wheel_x" value="0"/>
@@ -112,5 +112,5 @@
                 <cylinder length="${r_wheel_length}" radius="${r_wheel_radius}"/>
             </geometry>
-            <material name="blue"/>
+            <material name="red"/>
         </visual>
         <collision>
@@ -123,39 +123,85 @@
         </xacro:inertial_cylinder>
     </link>
-    <xacro:property name="c_wheel_joint_x" value="0.24"/>
-    <xacro:property name="c_wheel_joint_y" value="0"/>
-    <xacro:property name="c_wheel_joint_z" value="0"/>
-    <xacro:property name="c_wheel_joint_roll" value="0"/>
-    <xacro:property name="c_wheel_joint_pitch" value="0"/>
-    <xacro:property name="c_wheel_joint_yaw" value="0"/>
-    <!-- CASTER WHEEL -->
-    <joint name="caster_wheel_joint" type="fixed">
-        <parent link="chassis"/>
-        <child link="caster_wheel"/>
-        <origin xyz="${c_wheel_joint_x} ${c_wheel_joint_y} ${c_wheel_joint_z}" rpy="${c_wheel_joint_roll} ${c_wheel_joint_pitch} ${c_wheel_joint_yaw}"/>
-    </joint>
-    <xacro:property name="c_wheel_radius" value="0.05"/>
-    <xacro:property name="c_wheel_mass" value="0.1"/>
-    <xacro:property name="c_wheel_x" value="0"/>
-    <xacro:property name="c_wheel_y" value="0"/>
-    <xacro:property name="c_wheel_z" value="0"/>
-    <xacro:property name="c_wheel_roll" value="0"/>
-    <xacro:property name="c_wheel_pitch" value="0"/>
-    <xacro:property name="c_wheel_yaw" value="0"/>
-    <link name="caster_wheel">
-        <visual>
-            <geometry>
-                <sphere radius="${c_wheel_radius}"/>
-            </geometry>
-            <material name="black"/>
-        </visual>
-        <collision>
-            <geometry>
-                <sphere radius="${c_wheel_radius}"/>
-            </geometry>
-        </collision>
-        <xacro:inertial_sphere mass="${c_wheel_mass}" radius="${c_wheel_radius}">
-            <origin xyz="${c_wheel_x} ${c_wheel_y} ${c_wheel_z}" rpy="${c_wheel_roll} ${c_wheel_pitch} ${c_wheel_yaw}"/>
-        </xacro:inertial_sphere>
+    <!-- LEFT WHEEL1 -->
+    <joint name="left_wheel_joint1" type="continuous">
+        <parent link="base_link"/>
+        <child link="left_wheel1"/>
+        <origin xyz="-0.25 ${l_wheel_joint_y} ${l_wheel_joint_z}" rpy="${l_wheel_joint_roll} ${l_wheel_joint_pitch} ${l_wheel_joint_yaw}" />
+        <axis xyz="${l_wheel_joint_ax} ${l_wheel_joint_ay} ${l_wheel_joint_az}"/>
+    </joint>
+    <link name="left_wheel1">
+        <visual>
+            <geometry>
+                <cylinder length="${l_wheel_length}" radius="${l_wheel_radius}"/>
+            </geometry>
+            <material name="red"/>
+        </visual>
+        <collision>
+            <geometry>
+                <cylinder length="${l_wheel_length}" radius="${l_wheel_radius}"/>
+            </geometry>
+        </collision>
+        <xacro:inertial_cylinder mass="${l_wheel_m}" length="${l_wheel_length}" radius="${l_wheel_radius}">
+            <origin xyz="${l_wheel_x} ${l_wheel_y} ${l_wheel_z}" rpy="${l_wheel_roll} ${l_wheel_pitch} ${l_wheel_yaw}"/>
+        </xacro:inertial_cylinder>
+    </link>
+    <!-- RIGHT WHEEL1 -->
+    <joint name="right_wheel_joint1" type="continuous">
+        <parent link="base_link"/>
+        <child link="right_wheel1"/>
+        <origin xyz="-0.25 ${r_wheel_joint_y} ${r_wheel_joint_z}" rpy="${r_wheel_joint_roll} ${r_wheel_joint_pitch} ${r_wheel_joint_yaw}" />
+        <axis xyz="${r_wheel_joint_ax} ${r_wheel_joint_ay} ${r_wheel_joint_az}"/>
+    </joint>
+    <link name="right_wheel1">
+        <visual>
+            <geometry>
+                <cylinder length="${r_wheel_length}" radius="${r_wheel_radius}"/>
+            </geometry>
+            <material name="red"/>
+        </visual>
+        <collision>
+            <geometry>
+                <cylinder length="${r_wheel_length}" radius="${r_wheel_radius}"/>
+            </geometry>
+        </collision>
+        <xacro:inertial_cylinder mass="${r_wheel_m}" length="${r_wheel_length}" radius="${r_wheel_radius}">
+            <origin xyz="${r_wheel_x} ${r_wheel_y} ${r_wheel_z}" rpy="${r_wheel_roll} ${r_wheel_pitch} ${r_wheel_yaw}"/>
+        </xacro:inertial_cylinder>
+    </link>
+    <xacro:property name="robo_hub_joint_x" value="0"/>
+    <xacro:property name="robo_hub_joint_y" value="0"/>
+    <xacro:property name="robo_hub_joint_z" value="0"/>
+    <joint name="robo_hub_joint" type="fixed">
+        <parent link="base_link"/>
+        <child link="robo_hub"/>
+        <origin xyz="${robo_hub_joint_x} ${robo_hub_joint_y} ${robo_hub_joint_z}"/>
+    </joint>
+    <xacro:property name="robo_hub_x" value="0.1"/>
+    <xacro:property name="robo_hub_y" value="0"/>
+    <xacro:property name="robo_hub_z" value="0.4"/>
+    <xacro:property name="robo_hub_l" value="0.4"/>
+    <xacro:property name="robo_hub_w" value="0.3"/>
+    <xacro:property name="robo_hub_h" value="0.2"/>
+    <xacro:property name="robo_hub_roll" value="0"/>
+    <xacro:property name="robo_hub_pitch" value="0"/>
+    <xacro:property name="robo_hub_yaw" value="0"/>
+    <xacro:property name="robo_hub_m" value="0.5"/>
+    <link name="robo_hub">
+        <visual>
+            <origin xyz="${robo_hub_x} ${robo_hub_y} ${robo_hub_z}"/>
+            <geometry>
+                <box size="${robo_hub_w} ${robo_hub_l} ${robo_hub_h}"/>
+            </geometry>
+            <material name="green"/>
+        </visual>
+        <collision>
+            <origin xyz="${robo_hub_x} ${robo_hub_y} ${robo_hub_z}" rpy="${robo_hub_roll} ${robo_hub_pitch} ${robo_hub_yaw}"/>
+            <geometry>
+                <box size="${robo_hub_w} ${robo_hub_l} ${robo_hub_h}"/>
+            </geometry>
+        </collision>
+        <xacro:inertial_box mass="${robo_hub_m}" x="${robo_hub_w}" y="${robo_hub_l}" z="${robo_hub_h}">
+            <origin xyz="${robo_hub_x} ${robo_hub_y} ${robo_hub_z}" rpy="${robo_hub_roll} ${robo_hub_pitch} ${robo_hub_yaw}"/>
+        </xacro:inertial_box>
     </link>
 </robot>
