Commit message: ex 5.2 done

File: src/lab05/description/depth_camera.xacro (robot description, xacro)
@@ -4,10 +4,10 @@
         <parent link="chassis"/>
         <child link="camera_link"/>
-        <origin xyz="0.305 0 0.08" rpy="0 0 0"/>
+        <origin xyz="0.1 0 0.40" rpy="0 0 0"/>
     </joint>
     <link name="camera_link">
         <visual>
             <geometry>
-                <box size="0.010 0.03 0.03"/>
+                <cylinder length="0.5" radius="0.05"/>
             </geometry>
             <material name="red"/>

File: src/lab05/description/robot.urdf (robot description, URDF)
Before this commit: robot robot, 8 links, 7 joints
Links:
- link camera_link: geometry visual cylinder length=0.5 radius=0.05
Joints:
- joint camera_joint: origin xyz=0.305 0 0.08 rpy=0 0 0 -> xyz=0.1 0 0.40 rpy=0 0 0

Commit message: ex 3 done

File: src/lab05/description/depth_camera.xacro (robot description, xacro)
@@ -13,4 +13,9 @@
             <material name="red"/>
         </visual>
+        <collision>
+            <geometry>
+                <cylinder length="0.5" radius="0.05"/>
+            </geometry>
+        </collision>
     </link>
     <joint name="camera_optical_joint" type="fixed">

File: src/lab05/description/gazebo.xacro (robot description, xacro)
@@ -32,3 +32,11 @@
         </plugin>
     </gazebo>
+    <gazebo reference="chassis">
+        <sensor name="imu_sensor" type="imu">
+            <always_on>1</always_on>
+            <update_rate>1</update_rate>
+            <visualize>true</visualize>
+            <topic>imu</topic>
+        </sensor>
+    </gazebo>
 </robot>

File: src/lab05/description/robot.urdf (robot description, URDF)
Before this commit: robot robot, 8 links, 7 joints
Links:
- link camera_link: geometry collision cylinder length=0.5 radius=0.05; visual cylinder length=0.5 radius=0.05
- link caster_wheel: mass 0.1 -> 0.15

File: src/lab05/description/robot_core.xacro (robot description, xacro)
@@ -136,5 +136,5 @@
     </joint>
     <xacro:property name="c_wheel_radius" value="0.05"/>
-    <xacro:property name="c_wheel_mass" value="0.1"/>
+    <xacro:property name="c_wheel_mass" value="0.15"/>
     <xacro:property name="c_wheel_x" value="0"/>
     <xacro:property name="c_wheel_y" value="0"/>
